File: rusty_keys_comp.kicad_pcb (KiCad board)
At the start: 2 copper layers, 99.1 x 53.3 mm, 15 parts, among them J1 Conn_01x03_Pin, SW1 SW_Push, SW2 SW_Push, SW3 SW_Push, SW4 SW_Push, SW5 SW_Push, SW6 SW_Push

Commit message: ロゴ削除
Parts:
- removed REF**: RustyKeys_Logo, Bracket_Computer_Logo:RustyKeys_Logo
